Commit message: sample urdf of bot

File: jetbot/urdf/lidar.xacro (robot description, xacro)
@@ -2,7 +2,7 @@
 <robot xmlns:xacro="http://www.ros.org/wiki/xacro" >
     <joint name="laser_joint" type="fixed">
-        <parent link="chassis"/>
+        <parent link="base_link"/>
         <child link="laser_frame"/>
-        <origin xyz="0.1 0 0.175" rpy="0 0 0"/>
+        <origin xyz="0 0 0.26" rpy="0 0 0"/>
     </joint>
     <link name="laser_frame">
@@ -18,9 +18,7 @@
             </geometry>
         </collision>
-        <xacro:inertial_cylinder mass="0.1" length="0.04" radius="0.05">
-            <origin xyz="0 0 0" rpy="0 0 0"/>
-        </xacro:inertial_cylinder>
+        <xacro:cylinder_inertia m="0.1" r="0.05" h="0.04" xyz="0 0 0" rpy="0 0 0" />
     </link>
-    <gazebo reference="laser_frame">
+    <!-- <gazebo reference="laser_frame">
         <material>Gazebo/Red</material>
         <sensor name="laser" type="ray">
@@ -49,4 +47,4 @@
             </plugin>
         </sensor>
-    </gazebo>
+    </gazebo> -->
 </robot>

File: jetbot/urdf/robot.urdf.xacro (robot description, xacro)
@@ -3,3 +3,4 @@
     <xacro:include filename="common_properties.xacro" />
     <xacro:include filename="robot_core.xacro" />
+    <xacro:include filename="lidar.xacro" />
 </robot>

File: jetbot/urdf/robot_core.xacro (robot description, xacro)
@@ -45,5 +45,5 @@
     <xacro:wheel_link prefix="right" />
     <xacro:wheel_link prefix="left" />
-    <!-- <link name="caster_wheel_link">
+    <link name="caster_wheel_link">
         <visual>
             <geometry>
@@ -61,5 +61,5 @@
         <xacro:sphere_inertia m="0.5" r="${2*wheel_radius / 2.0}"
                               xyz="0 0 0" rpy="0 0 0" />
-    </link> -->
+    </link>
     <joint name="base_joint" type="fixed">
         <parent link="base_footprint" />
@@ -70,5 +70,5 @@
         <parent link="base_link" />
         <child link="right_wheel_link" />
-        <origin xyz="0 ${-(base_width + wheel_length) / 2.0} 0" rpy="0 0 0" />
+        <origin xyz="-0.23 ${-(base_width + wheel_length) / 2.0} 0" rpy="0 0 0" />
         <axis xyz="0 1 0" />
     </joint>
@@ -76,12 +76,12 @@
         <parent link="base_link" />
         <child link="left_wheel_link" />
-        <origin xyz="0 ${(base_width + wheel_length) / 2.0} 0" rpy="0 0 0" />
+        <origin xyz="-0.23 ${(base_width + wheel_length) / 2.0} 0" rpy="0 0 0" />
         <axis xyz="0 1 0" />
     </joint>
-    <!-- <joint name="base_caster_wheel_joint" type="fixed">
+    <joint name="base_caster_wheel_joint" type="fixed">
         <parent link="base_link" />
         <child link="caster_wheel_link" />
         <origin xyz="${base_length / 3.0} 0 ${-wheel_radius / 2.0}" rpy="0 0 0" />
-    </joint> -->
+    </joint>
     <!-- Gazebo tags -->
     <!-- <gazebo reference="base_link">
